File: board/board.kicad_pcb (KiCad board)
At the start: 2 copper layers, 21 x 13 mm, 1 part

Commit message: initial
Parts:
- added C1: 100nF, Capacitor_SMD:C_0603_1608Metric, F.Cu at (235.2, 109.6)
- added C2: 100nF, Capacitor_SMD:C_0603_1608Metric, F.Cu at (218.9, 109.8)
- added C3: 100nF, Capacitor_SMD:C_0603_1608Metric, F.Cu at (252.5, 109.8)
- added J1: 007_ADC, on_edge:on_edge_2x05_device, F.Cu at (200.0, 86.5)
- added J2: VP0365540000G, b129:VP0365540000G, F.Cu at (248.8, 95.8)
- added J3: VP0365540000G, b129:VP0365540000G, F.Cu at (248.8, 123.6)
- added J4: 007_ADC, on_edge:on_edge_2x05_device, F.Cu at (200.0, 102.5)
- added R1: 10k, Capacitor_SMD:C_0603_1608Metric, F.Cu at (216.7, 110.5)
- added R2: 10k, Capacitor_SMD:C_0603_1608Metric, F.Cu at (216.7, 109.0)
- added U1: ACS733KLATR-65AB-T, b129:SOIC-16W_6.5x12.8mm_P1.27mm, F.Cu at (241.9, 109.7)
- added U2: ACS733KLATR-65AB-T, b129:SOIC-16W_6.5x12.8mm_P1.27mm, F.Cu at (225.7, 109.5)
- added U3: ACS733KLATR-65AB-T, b129:SOIC-16W_6.5x12.8mm_P1.27mm, F.Cu at (259.2, 109.6)
- moved LOGO1 78.3 mm to (227.5, 87.5)
Routing:
- net GND: track 0.00 -> 109.2 mm, vias 0 -> 4
- net /hall/VCC: track 0.00 -> 94.4 mm, vias 0 -> 4
- net /hall2/VIOUT: track 0.00 -> 64.5 mm, vias 0 -> 2
- net /hall/VIOUT: track 0.00 -> 45.9 mm, vias 0 -> 2
- net Net-(J1-Pad4): track 0.00 -> 44.8 mm, vias 0 -> 2
- net /hall2/I-: track 0.00 -> 30.7 mm
- net /hall2/I+: track 0.00 -> 30.1 mm
- net /hall1/I-: track 0.00 -> 29.6 mm
- net /hall/I+: track 0.00 -> 26.5 mm
- net /hall/I-: track 0.00 -> 26.4 mm
- net /hall1/VIOUT: track 0.00 -> 24.3 mm, vias 0 -> 2
- net /hall1/I+: track 0.00 -> 23.6 mm
- net Net-(J1-Pad10): track 0.00 -> 22.4 mm, vias 0 -> 2
Other:
- board size 21 x 13 mm -> 69 x 61 mm
- board text added: "osf.007"
- board text added: "osf.b129.v1.0"
